Commit message: update-lab3

File: src/dobot/urdf/dobot.urdf (robot description, URDF)
Before this commit: robot dobot, 5 links, 4 joints
Links:
- added link fourth; visual box size=0.06 0.06 0.06
- link gripper: geometry visual box size=0.06 0.03 0.09
Joints:
- added joint joint5: type revolute, parent arm2, child fourth, origin xyz=0.0 0.0 0.147, axis 0 1 0, limit lower=-1.571 upper=1.571 effort=${params.effort} velocity=${params.joint3_velocity[0]}
- joint joint1: limit lower=${params.joint1_limits[0]} upper=${params.joint1_limits[1]} effort=${params.effort} velocity=${params.joint1_velocity[0]} -> lower=${params.joint1_limits[1]} upper=${params.joint1_limits[0]} effort=${params.effort} velocity=${params.joint1_velocity[0]}
- joint joint3: limit lower=${params.joint3_limits[0]} upper=${params.joint3_limits[1]} effort=${params.effort} velocity=${params.joint3_velocity[0]} -> lower=${params.joint3_limits[1]} upper=${params.joint3_limits[0]} effort=${params.effort} velocity=${params.joint3_velocity[0]}
- joint joint4: axis ${params.joint4_axis} -> 1 0 0; limit lower=${params.joint4_limits[0]} upper=${params.joint4_limits[1]} effort=${params.effort} velocity=${params.joint4_velocity[0]} -> lower=${params.joint4_limits[1]} upper=${params.joint4_limits[0]} effort=${params.effort} velocity=${params.joint4_velocity[0]}; origin xyz=${params.joint4_origins} -> xyz=0.03 0.0 0.03; parent arm2 -> fourth

Commit message: refaktoryzacja kodu po lab3

File: src/dobot/urdf/dobot.urdf (robot description, URDF)
Before this commit: robot dobot, 6 links, 5 joints
Links:
- link fourth: geometry visual box size=${params.fourth_size}
- link gripper: geometry visual box size=${params.gripper_size}
Joints:
- joint joint4: axis 1 0 0 -> ${params.joint4_axis}; origin xyz=0.03 0.0 0.03 -> xyz=${params.joint4_origins}
- joint joint5: axis 0 1 0 -> ${params.joint5_axis}; limit lower=-1.571 upper=1.571 effort=${params.effort} velocity=${params.joint3_velocity[0]} -> lower=${params.joint5_limits[0]} upper=${params.joint5_limits[1]} effort=${params.effort} velocity=${params.joint3_velocity[0]}; origin xyz=0.0 0.0 0.147 -> xyz=${params.joint5_origins}
