Commit message: laby_5

File: src/dobot/urdf/dobot2.urdf (robot description, URDF)
Before this commit: robot dobot, 8 links, 7 joints
Links:
- removed link camera
- added link camera_stick; visual box size=${params.camera_grip_size}
- link camera_link: geometry visual box size=${params.camera_size}
Joints:
- joint joint6: child camera_link -> camera_stick
- joint joint7: child camera -> camera_link; parent camera_link -> camera_stick
